File: kicad/nanov3.kicad_pcb (KiCad board)
At the start: 2 copper layers, 16 parts, among them J1 RJ45, P1 SUPP32, U1 4N33, U2 4N33

Commit message: новая плата
Parts:
- added D3: LED, LEDs:LED-5MM, F.Cu at (107.7, 66.0)
- added D4: LED, LEDs:LED-5MM, F.Cu at (107.7, 58.4)
- added P2: CONN_01X03, Connect:Wafer_Horizontal10x5.8x7RM2.5-3, F.Cu at (102.9, 44.5)
- added R11: 5k, Discret:R4, F.Cu at (99.1, 71.8)
- added R12: 5k, Discret:R4, F.Cu at (101.6, 73.7)
- added R13: 200, Discret:R4, F.Cu at (99.1, 55.2)
- added R14: 200, Discret:R4, F.Cu at (101.6, 56.5)
- added SP1: SPEAKER, Buzzers_Beepers:BUZZER, F.Cu at (63.5, 35.6)
- added SW1: SW_PUSH, Buttons_Switches_ThroughHole:SW_Tactile_SPST_Angled, F.Cu at (109.2, 45.7)
- added SW2: SW_PUSH, Buttons_Switches_ThroughHole:SW_Tactile_SPST_Angled, F.Cu at (109.2, 71.1)
Routing:
- net Net-(D3-Pad2): track 70.1 -> 197.1 mm
- net Net-(P1-Pad13): track 0.00 -> 72.7 mm
- net Net-(P1-Pad9): track 0.00 -> 49.7 mm
- net Net-(P1-Pad29): track 27.1 -> 74.8 mm
- net Net-(P1-Pad15): track 0.00 -> 40.2 mm
- net Net-(P1-Pad14): track 0.00 -> 39.8 mm
- net Net-(P1-Pad18): track 0.00 -> 25.5 mm
- net Net-(D3-Pad1): track 0.00 -> 19.5 mm
- net Net-(P1-Pad32): track 0.00 -> 14.5 mm
- net Net-(D4-Pad1): track 0.00 -> 10.1 mm
- net Net-(P1-Pad31): track 0.00 -> 8.44 mm
- net Net-(P1-Pad8): track 0.00 -> 4.06 mm
- net Net-(P1-Pad7): track 0.00 -> 4.06 mm
- net Net-(P1-Pad6): track 0.00 -> 4.06 mm
- net Net-(P1-Pad5): track 0.00 -> 4.06 mm
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- added copper zone on B.Cu, net Net-(D1-Pad1)
- added copper zone on B.Cu, net Net-(D3-Pad2)
- added copper zone on B.Cu, net Net-(J1-Pad1)
- added copper zone on B.Cu, net Net-(J1-Pad7)
- added copper zone on B.Cu, net Net-(P1-Pad15)
- added copper zone on B.Cu, net Net-(P1-Pad31)
- added copper zone on B.Cu, net Net-(P1-Pad32)
- added copper zone on B.Cu, net Net-(P1-Pad9)
- added copper zone on B.Cu, net Net-(R1-Pad1)
- added copper zone on B.Cu, net Net-(R1-Pad2)
